Commit message: changes

File: src/segmentation/urdf/camera.urdf (robot description, URDF)
Before this commit: robot camera, 4 links, 3 joints
Joints:
- joint world_to_base: type fixed -> continuous

Commit message: spawned camera with transparent link

File: src/segmentation/urdf/camera.urdf (robot description, URDF)
Before this commit: robot camera, 4 links, 3 joints
Links:
- added link base_link, mass 1e-5; collision box size=0.1 0.1 1; visual box size=0.1 0.1 1
- added link link1, mass 1e-5; collision box size=0.1 0.1 1; visual box size=0.1 0.1 1
Joints:
- added joint joint1: type continuous, parent base_link, child link1, origin xyz=0 0.1 1.95 rpy=0 1.5708 0, axis 1 0 0
- added joint joint2: type fixed, parent link1, child camera_link, origin xyz=0 0.1 0.9 rpy=0 0 0
- joint world_to_base: child camera_link -> base_link; type continuous -> fixed
