Commit message: removed prefix

File: src/segmentation/gazebo/camera.gazebo.xacro (robot description, xacro)
@@ -5,5 +5,5 @@
 -->
 <robot xmlns:xacro="http://ros.org/wiki/xacro">
-  <xacro:macro name="camera_gazebo" params="prefix">
+  <xacro:macro name="camera_gazebo">
     <!-- ros_control plugin -->
     <gazebo>
@@ -13,9 +13,9 @@
     </gazebo>
     <!-- Link1 -->
-    <gazebo reference="${prefix}base_link">
+    <gazebo reference="base_link">
       <material>Gazebo/GreyTransparent</material>
     </gazebo>
     <!-- Link2 -->
-    <gazebo reference="${prefix}link1">
+    <gazebo reference="link1">
       <mu1>0.2</mu1>
       <mu2>0.2</mu2>
@@ -23,5 +23,5 @@
     </gazebo>
     <!-- camera_link -->
-    <gazebo reference="${prefix}camera_link">
+    <gazebo reference="camera_link">
       <mu1>0.2</mu1>
       <mu2>0.2</mu2>
@@ -29,5 +29,5 @@
     </gazebo>
     <!-- hokuyo -->
-    <gazebo reference="${prefix}hokuyo_link">
+    <gazebo reference="hokuyo_link">
       <sensor type="gpu_ray" name="head_hokuyo_sensor">
         <pose>0 0 0 0 0 0</pose>
@@ -64,5 +64,5 @@
       </sensor>
     </gazebo>
-    <gazebo reference="${prefix}camera_link">
+    <gazebo reference="camera_link">
         <sensor type="depth" name="realsense">
 	        <always_on>1</always_on>
@@ -108,5 +108,5 @@
     </gazebo>
     <!-- camera -->
-    <!-- <gazebo reference="${prefix}camera_link">
+    <!-- <gazebo reference="camera_link">
       <sensor type="camera" name="camera1">
         <update_rate>30.0</update_rate>

File: src/segmentation/ros2_control/camera.ros2_control.xacro (robot description, xacro)
@@ -1,10 +1,10 @@
 <?xml version="1.0"?>
 <robot xmlns:xacro="http://www.ros.org/wiki/xacro">
-  <xacro:macro name="camera_ros2_control" params="name prefix">
+  <xacro:macro name="camera_ros2_control" params="name">
     <ros2_control name="${name}" type="system">
       <hardware>
           <plugin>gazebo_ros2_control/GazeboSystem</plugin>
       </hardware>
-      <joint name="${prefix}joint1">
+      <joint name="joint1">
         <command_interface name="position">
           <param name="min">-10</param>

File: src/segmentation/urdf/camera.urdf.xacro (robot description, xacro)
@@ -1,5 +1,5 @@
 <?xml version="1.0"?>
 <robot xmlns:xacro="http://www.ros.org/wiki/xacro">
-  <xacro:macro name="camera" params="parent prefix *origin">
+  <xacro:macro name="camera" params="parent *origin">
   <!-- Constants for robot dimensions -->
   <xacro:property name="mass" value="1" /> <!-- arbitrary value for mass -->
@@ -10,11 +10,11 @@
   <xacro:property name="camera_link" value="0.05" /> <!-- Size of square 'camera' box -->
   <xacro:property name="axel_offset" value="0.05" /> <!-- Space btw top of beam and the each joint -->
-  <joint name="${prefix}base_joint" type="fixed">
+  <joint name="base_joint" type="fixed">
     <xacro:insert_block name="origin" />
     <parent link="${parent}"/>
-    <child link="${prefix}base_link" />
+    <child link="base_link" />
   </joint>
   <!-- Base Link -->
-  <link name="${prefix}base_link">
+  <link name="base_link">
     <!-- <collision>
       <origin xyz="0 0 ${height1/2}" rpy="0 0 0"/>
@@ -39,7 +39,7 @@
       </inertial>
     </link>
-    <joint name="${prefix}joint1" type="continuous">
-      <parent link="${prefix}base_link"/>
-      <child link="${prefix}link1"/>
+    <joint name="joint1" type="continuous">
+      <parent link="base_link"/>
+      <child link="link1"/>
       <origin xyz="0 ${width} ${height1 - axel_offset}" rpy="0 1.5708 0"/>
       <axis xyz="1 0 0"/>
@@ -47,5 +47,5 @@
     </joint>
     <!-- Middle Link -->
-    <link name="${prefix}link1">
+    <link name="link1">
       <collision>
         <origin xyz="0 0 ${height2/2 - axel_offset}" rpy="0 0 0"/>
@@ -70,7 +70,7 @@
         </inertial>
       </link>
-      <!-- <joint name="${prefix}joint2" type="continuous">
-        <parent link="${prefix}link1"/>
-        <child link="${prefix}link2"/>
+      <!-- <joint name="joint2" type="continuous">
+        <parent link="link1"/>
+        <child link="link2"/>
         <origin xyz="0 ${width} ${height2 - axel_offset*2}" rpy="0 0 0"/>
         <axis xyz="1 0 0"/>
@@ -78,5 +78,5 @@
       </joint> -->
       <!-- Top Link -->
-      <!-- <link name="${prefix}link2">
+      <!-- <link name="link2">
         <collision>
           <origin xyz="0 0 ${height3/2 - axel_offset}" rpy="0 0 0"/>
@@ -101,20 +101,20 @@
           </inertial>
         </link> -->
-        <joint name="${prefix}tool_joint" type="fixed">
+        <joint name="tool_joint" type="fixed">
           <origin xyz="0 0 1" rpy="0 0 0" />
-          <parent link="${prefix}link1"/>
-          <child link="${prefix}tool_link" />
+          <parent link="link1"/>
+          <child link="tool_link" />
         </joint>
         <!-- Tool Link -->
-        <link name="${prefix}tool_link">
+        <link name="tool_link">
         </link>
-        <joint name="${prefix}hokuyo_joint" type="fixed">
+        <joint name="hokuyo_joint" type="fixed">
           <axis xyz="0 1 0" />
           <origin xyz="0 0 ${height3 - axel_offset/2}" rpy="0 0 0"/>
-          <parent link="${prefix}link1"/>
-          <child link="${prefix}hokuyo_link"/>
+          <parent link="link1"/>
+          <child link="hokuyo_link"/>
         </joint>
         <!-- Hokuyo Laser -->
-        <link name="${prefix}hokuyo_link">
+        <link name="hokuyo_link">
           <collision>
             <origin xyz="0 0 0" rpy="0 0 0"/>
@@ -135,12 +135,12 @@
           </inertial>
         </link>
-        <joint name="${prefix}camera_joint" type="fixed">
+        <joint name="camera_joint" type="fixed">
           <axis xyz="0 1 0" />
           <origin xyz="${camera_link} 0 ${height3 - axel_offset*2}" rpy="0 0 0"/>
-          <parent link="${prefix}link1"/>
-          <child link="${prefix}camera_link"/>
+          <parent link="link1"/>
+          <child link="camera_link"/>
         </joint>
         <!-- Camera -->
-        <link name="${prefix}camera_link">
+        <link name="camera_link">
           <collision>
             <origin xyz="0 0 0" rpy="0 0 0"/>
@@ -164,12 +164,12 @@
         <!-- generate an optical frame http://www.ros.org/reps/rep-0103.html#suffix-frames
         so that ros and opencv can operate on the camera frame correctly -->
-        <joint name="${prefix}camera_optical_joint" type="fixed">
+        <joint name="camera_optical_joint" type="fixed">
           <!-- these values have to be these values otherwise the gazebo camera image
           won't be aligned properly with the frame it is supposedly originating from -->
           <origin xyz="0 0 0" rpy="${-pi/2} 0 ${-pi/2}"/>
-          <parent link="${prefix}camera_link"/>
-          <child link="${prefix}camera_link_optical"/>
+          <parent link="camera_link"/>
+          <child link="camera_link_optical"/>
         </joint>
-        <link name="${prefix}camera_link_optical">
+        <link name="camera_link_optical">
         </link>
   </xacro:macro>

File: src/segmentation/urdf/rbot.urdf.xacro (robot description, xacro)
@@ -20,9 +20,9 @@
     <static>true</static>
   </gazebo>
-  <xacro:camera parent="world" prefix="$(arg prefix)">
+  <xacro:camera parent="world">
     <origin xyz="0 0 0" rpy="0 0 0" />
   </xacro:camera>
-  <xacro:camera_gazebo prefix="$(arg prefix)" />
+  <xacro:camera_gazebo />
   <xacro:camera_ros2_control
-    name="CAMERA" prefix="$(arg prefix)" />
+    name="CAMERA"/>
 </robot>
